Commit message: Cup positie
Cup op juiste positie gezet

File: urdf/cup.urdf (robot description, URDF)
Before this commit: robot cup, 1 links, 0 joints
Links:
- link base_link: geometry visual cylinder length=0.08 radius=0.02

Commit message: mok gripping werk soortvan wip

File: urdf/cup.urdf (robot description, URDF)
Before this commit: robot cup, 1 links, 0 joints
Links:
- removed link base_link
- added link cup_link; visual cylinder length=0.08 radius=0.02

Commit message: werkt bijna

File: urdf/cup.urdf (robot description, URDF)
Before this commit: robot cup, 1 links, 0 joints
Links:
- link cup_link: geometry visual cylinder length=0.08 radius=0.015
